File: PID-controller-pcb/PID-controller-pcb.sch (KiCad schematic (older format))
At the start: 8 parts

Commit message: updated schematic and pcb pdfs
Parts:
- added SW?: SW_DPDT_x2, symbol Switch:SW_DPDT_x2
- added U?: BeagleSpyConnector, symbol New_Library:BeagleSpyConnector
Connections:
- net 3V3: now also SW?.3 (C)
- net BNC3: now also U?.8 (A1); no longer U?.7 (A0)
- net GND: now also SW?.1 (A), U?.10 (GND), U?.2 (GND); no longer J?.2 (Ext1), J?.2 (Ext1), J?.2 (Ext1), U?.2 (GND)
- net MISO: now also U?.5 (MISO)
- net MOSI: now also U?.8 (MOSI)
- net SCL: now also U?.1 (SCL)
- net SCLK: now also U?.7 (SCLK)
- net SDA: now also U?.3 (SDA)
- net nSS: now also U?.9 (SS)
- net SW1: now reaches U?.1 (GPIO0)
- net AGND: now reaches U?.9 (A2)
- net AGND: now also J?.2 (Ext1), J?.2 (Ext1), J?.2 (Ext1), U?.2 (GND), U?.7 (A0)
- new net GP00: SW?.2 (B)
Other:
- moved on the sheet: J?A
Changed lines of the file:
@@
 L Connector:Conn_Coaxial_x2_Isolated J?
 U 1 1 60D4852C
-P 8300 1000
-F 0 "J?" H 8400 975 50  0000 L CNN
-F 1 "CurrOut_BNC" H 8400 884 50  0000 L CNN
-F 2 "" H 8300 1000 50  0001 C CNN
-F 3 " ~" H 8300 1000 50  0001 C CNN
-	1    8300 1000
+P 3500 950
+F 0 "J?" H 3600 925 50  0000 L CNN
+F 1 "CurrOut_BNC" H 3600 834 50  0000 L CNN
+F 2 "" H 3500 950 50  0001 C CNN
+F 3 " ~" H 3500 950 50  0001 C CNN
+	1    3500 950
 	1    0    0    -1
 $EndComp
@@
 SCL
 Text GLabel 6450 3500 1    50   Input ~ 0
-GND
+AGND
 Text GLabel 6550 3500 1    50   Input ~ 0
 BNC1
@@
 Wire Wire Line
 	6550 3500 6550 3600
-Text GLabel 8100 1300 3    50   Input ~ 0
+Text GLabel 3300 1250 3    50   Input ~ 0
 DAC_OUT
 Wire Wire Line
-	8100 1000 8100 1300
-Text GLabel 8300 1300 3    50   Input ~ 0
-GND
+	3300 950  3300 1250
+Text GLabel 3500 1250 3    50   Input ~ 0
+AGND
 Text GLabel 9100 1300 3    50   Input ~ 0
-GND
+AGND
 Text GLabel 9950 1300 3    50   Input ~ 0
-GND
+AGND
 Wire Wire Line
 	9100 1300 9100 1200
@@
 Text GLabel 7250 3500 1    50   Input ~ 0
 BNC2
-Text GLabel 7550 3500 1    50   Input ~ 0
+Text GLabel 7450 3500 1    50   Input ~ 0
 BNC3
 Text GLabel 7750 3500 1    50   Input ~ 0
 GND
-NoConn ~ 7350 3600
-NoConn ~ 7450 3600
-NoConn ~ 7650 3600
 Text GLabel 7850 3500 1    50   Input ~ 0
 SDA
@@
 	7250 3500 7250 3600
 Wire Wire Line
-	7550 3500 7550 3600
+	7450 3500 7450 3600
 Wire Wire Line
 	7750 3500 7750 3600
@@
 	8150 3500 8150 3600
 Wire Wire Line
-	8300 1300 8300 1200
+	3500 1250 3500 1150
 Text GLabel 7700 2300 2    50   Input ~ 0
 SCL
@@
 Wire Wire Line
 	9050 3000 9200 3000
+Text GLabel 7550 3500 1    50   Input ~ 0
+AGND
+Wire Wire Line
+	7550 3500 7550 3600
+Text GLabel 7350 3500 1    50   Input ~ 0
+AGND
+Wire Wire Line
+	7350 3500 7350 3600
+NoConn ~ 7650 3600
+$Comp
+L Switch:SW_DPDT_x2 SW?
+U 1 1 60F7E6EA
+P 4450 2000
+F 0 "SW?" H 4450 2285 50  0000 C CNN
+F 1 "SW_DPDT_x2" H 4450 2194 50  0000 C CNN
+F 2 "" H 4450 2000 50  0001 C CNN
+F 3 "~" H 4450 2000 50  0001 C CNN
+	1    4450 2000
+	-1   0    0    -1
+$EndComp
+Text GLabel 6000 1000 0    50   Input ~ 0
+SW1
+Wire Wire Line
+	6000 1000 6100 1000
+Text GLabel 4800 2000 2    50   Input ~ 0
+GP00
+Wire Wire Line
+	4800 2000 4650 2000
+Text GLabel 4100 1900 0    50   Input ~ 0
+GND
+Wire Wire Line
+	4100 1900 4250 1900
+Text GLabel 4100 2100 0    50   Input ~ 0
+3V3
+Wire Wire Line
+	4100 2100 4250 2100
+$Comp
+L New_Library:BeagleSpyConnector U?
+U 1 1 60F87943
+P 4200 3100
+F 0 "U?" H 4200 3525 50  0000 C CNN
+F 1 "BeagleSpyConnector" H 4200 3434 50  0000 C CNN
+F 2 "" H 4200 3550 50  0001 C CNN
+F 3 "" H 4200 3550 50  0001 C CNN
+	1    4200 3100
+	-1   0    0    -1
+$EndComp
+Text GLabel 4750 3300 2    50   Input ~ 0
+SCL
+Text GLabel 4750 3200 2    50   Input ~ 0
+SDA
+Text GLabel 4750 3100 2    50   Input ~ 0
+MISO
+Text GLabel 4750 3000 2    50   Input ~ 0
+SCLK
+Text GLabel 4750 2900 2    50   Input ~ 0
+nSS
+Text GLabel 3650 3300 0    50   Input ~ 0
+GND
+Text GLabel 3650 3000 0    50   Input ~ 0
+MOSI
+Text GLabel 3650 2900 0    50   Input ~ 0
+GND
+Wire Wire Line
+	3650 2900 3850 2900
+Wire Wire Line
+	3650 3000 3850 3000
+Wire Wire Line
+	3650 3300 3850 3300
+Wire Wire Line
+	4750 2900 4550 2900
+Wire Wire Line
+	4750 3000 4550 3000
+Wire Wire Line
+	4750 3100 4550 3100
+Wire Wire Line
+	4750 3200 4550 3200
+Wire Wire Line
+	4750 3300 4550 3300
+NoConn ~ 3850 3100
+NoConn ~ 3850 3200
 $EndSCHEMATC
